Commit message: updated joint state pub for robot visualization

File: g1_sdk/urdf/g1_23dof.urdf (robot description, URDF)
Before this commit: robot g1_23dof, 34 links, 33 joints
Links:
- link base_link: geometry visual mesh filename=package://g1_sdk/meshes/pelvis.STL
- link head_link: geometry collision mesh filename=package://g1_sdk/meshes/head_link.STL; visual mesh filename=package://g1_sdk/meshes/head_link.STL
- link left_ankle_pitch_link: geometry collision mesh filename=package://g1_sdk/meshes/left_ankle_pitch_link.STL; visual mesh filename=package://g1_sdk/meshes/left_ankle_pitch_link.STL
- link left_ankle_roll_link: geometry collision sphere radius=0.005; collision sphere radius=0.005
- link left_elbow_link: geometry collision mesh filename=package://g1_sdk/meshes/left_elbow_link.STL; visual mesh filename=package://g1_sdk/meshes/left_elbow_link.STL
- link left_hip_pitch_link: geometry collision mesh filename=package://g1_sdk/meshes/left_hip_pitch_link.STL; visual mesh filename=package://g1_sdk/meshes/left_hip_pitch_link.STL
- link left_hip_roll_link: geometry collision mesh filename=package://g1_sdk/meshes/left_hip_roll_link.STL; visual mesh filename=package://g1_sdk/meshes/left_hip_roll_link.STL
- link left_hip_yaw_link: geometry collision mesh filename=package://g1_sdk/meshes/left_hip_yaw_link.STL; visual mesh filename=package://g1_sdk/meshes/left_hip_yaw_link.STL
- link left_knee_link: geometry collision mesh filename=package://g1_sdk/meshes/left_knee_link.STL; visual mesh filename=package://g1_sdk/meshes/left_knee_link.STL
- link left_shoulder_pitch_link: geometry collision cylinder length=0.05 radius=0.03; visual mesh filename=package://g1_sdk/meshes/left_shoulder_pitch_link.STL
- link left_shoulder_roll_link: geometry collision cylinder length=0.03 radius=0.03; visual mesh filename=package://g1_sdk/meshes/left_shoulder_roll_link.STL
- link left_shoulder_yaw_link: geometry collision mesh filename=package://g1_sdk/meshes/left_shoulder_yaw_link.STL; visual mesh filename=package://g1_sdk/meshes/left_shoulder_yaw_link.STL
- link left_wrist_roll_rubber_hand: geometry collision mesh filename=package://g1_sdk/meshes/left_wrist_roll_rubber_hand.STL; visual mesh filename=package://g1_sdk/meshes/left_wrist_roll_rubber_hand.STL
- link logo_link: geometry collision mesh filename=package://g1_sdk/meshes/logo_link.STL; visual mesh filename=package://g1_sdk/meshes/logo_link.STL
- link pelvis_contour_link: geometry collision mesh filename=package://g1_sdk/meshes/pelvis_contour_link.STL; visual mesh filename=package://g1_sdk/meshes/pelvis_contour_link.STL
- link right_ankle_pitch_link: geometry collision mesh filename=package://g1_sdk/meshes/right_ankle_pitch_link.STL; visual mesh filename=package://g1_sdk/meshes/right_ankle_pitch_link.STL
- link right_ankle_roll_link: geometry collision sphere radius=0.005; collision sphere radius=0.005
- link right_elbow_link: geometry collision mesh filename=package://g1_sdk/meshes/right_elbow_link.STL; visual mesh filename=package://g1_sdk/meshes/right_elbow_link.STL
- link right_hip_pitch_link: geometry collision mesh filename=package://g1_sdk/meshes/right_hip_pitch_link.STL; visual mesh filename=package://g1_sdk/meshes/right_hip_pitch_link.STL
- link right_hip_roll_link: geometry collision mesh filename=package://g1_sdk/meshes/right_hip_roll_link.STL; visual mesh filename=package://g1_sdk/meshes/right_hip_roll_link.STL
- link right_hip_yaw_link: geometry collision mesh filename=package://g1_sdk/meshes/right_hip_yaw_link.STL; visual mesh filename=package://g1_sdk/meshes/right_hip_yaw_link.STL
- link right_knee_link: geometry collision mesh filename=package://g1_sdk/meshes/right_knee_link.STL; visual mesh filename=package://g1_sdk/meshes/right_knee_link.STL
- link right_shoulder_pitch_link: geometry collision cylinder length=0.05 radius=0.03; visual mesh filename=package://g1_sdk/meshes/right_shoulder_pitch_link.STL
- link right_shoulder_roll_link: geometry collision cylinder length=0.03 radius=0.03; visual mesh filename=package://g1_sdk/meshes/right_shoulder_roll_link.STL
- link right_shoulder_yaw_link: geometry collision mesh filename=package://g1_sdk/meshes/right_shoulder_yaw_link.STL; visual mesh filename=package://g1_sdk/meshes/right_shoulder_yaw_link.STL
- link right_wrist_roll_rubber_hand: geometry collision mesh filename=package://g1_sdk/meshes/right_wrist_roll_rubber_hand.STL; visual mesh filename=package://g1_sdk/meshes/right_wrist_roll_rubber_hand.STL
- link torso_link: geometry collision mesh filename=package://g1_sdk/meshes/torso_link.STL; visual mesh filename=package://g1_sdk/meshes/torso_link.STL
- link waist_support_link: geometry collision mesh filename=package://g1_sdk/meshes/waist_support_link.STL; visual mesh filename=package://g1_sdk/meshes/waist_support_link.STL
- link waist_yaw_fixed_link: geometry visual mesh filename=package://g1_sdk/meshes/waist_yaw_link.STL
